Commit message: 20250929

File: src/zlab_robot_description/urdf/zlab_robot.urdf.xacro (robot description, xacro)
@@ -1,293 +1,307 @@
 <?xml version="1.0" encoding="utf-8"?>
 <robot name="zlab_robot" xmlns:xacro="http://www.ros.org/wiki/xacro">
-	<!-- 机械臂实例化与配置参数 -->
-	<xacro:arg name="config_file" default="../../../config/robot_arms.yaml" />
-	<xacro:arg name="parent_link" default="world" />
-	<xacro:arg name="arm_id" default="zlab_arm" />
-	<xacro:arg name="default_prefix" default="" />
-	<xacro:arg name="base_xyz" default="0 0 0" />
-	<xacro:arg name="base_rpy" default="0 0 0" />
-	<xacro:property name="config_path" value="$(arg config_file)" />
-	<xacro:property name="resolved_config_path" value="${config_path}" />
-	<xacro:property name="robot_config" value="${xacro.load_yaml(resolved_config_path) or dict()}" />
-	<xacro:property name="arms_config" value="${robot_config.get('arms', dict())}" />
-	<xacro:property name="enabled_arms" value="${[(name, cfg) for name, cfg in arms_config.items() if cfg.get('enabled', False)]}" />
-	<xacro:property name="default_parent_link" value="$(arg parent_link)" />
-	<!-- 通用外观设置 -->
-	<xacro:property name="link_material" value="silver" />
-	<xacro:property name="link_color_rgba" value="0.89804 0.91765 0.92941 1" />
-	<!-- 可复用的带惯量链接定义 -->
-	<xacro:macro name="link_with_inertial" params="name xyz rpy mass ixx ixy ixz iyy iyz izz visual_mesh collision_mesh scale:='1 1 1'">
-		<link name="${name}">
-			<inertial>
-				<origin xyz="${xyz}" rpy="${rpy}" />
-				<mass value="${mass}" />
-				<inertia ixx="${ixx}" ixy="${ixy}" ixz="${ixz}" iyy="${iyy}" iyz="${iyz}" izz="${izz}" />
-			</inertial>
-			<visual>
-				<origin xyz="0 0 0" rpy="0 0 0" />
-				<geometry>
-					<mesh filename="${visual_mesh}" scale="${scale}" />
-				</geometry>
-						<material name="${link_material}">
-							<color rgba="${link_color_rgba}" />
-						</material>
-			</visual>
-			<collision>
-				<origin xyz="0 0 0" rpy="0 0 0" />
-				<geometry>
-					<mesh filename="${collision_mesh}" scale="${scale}" />
-				</geometry>
-			</collision>
-		</link>
-	</xacro:macro>
-	<xacro:macro name="instantiate_arms" params="arm_list">
-		<xacro:if value="${len(arm_list) > 0}">
-			<xacro:property name="arm_entry" value="${arm_list[0]}" />
-			<xacro:property name="arm_cfg" value="${arm_entry[1]}" />
-			<xacro:property name="arm_name" value="${arm_entry[0]}" />
-			<xacro:property name="arm_id" value="${arm_cfg.get('arm_id', arm_name)}" />
-			<xacro:property name="raw_prefix" value="${arm_cfg.get('prefix', arm_name)}" />
-			<xacro:property name="prefix" value="${raw_prefix if raw_prefix.endswith('_') else raw_prefix + '_'}" />
-			<xacro:property name="base_xyz_list" value="${arm_cfg.get('base_xyz', [0.0, 0.0, 0.0])}" />
-			<xacro:property name="base_rpy_list" value="${arm_cfg.get('base_rpy', [0.0, 0.0, 0.0])}" />
-			<xacro:property name="base_xyz_str" value="${' '.join([str(x) for x in base_xyz_list])}" />
-			<xacro:property name="base_rpy_str" value="${' '.join([str(x) for x in base_rpy_list])}" />
-			<xacro:property name="arm_parent_link" value="${arm_cfg.get('parent_link', '')}" />
-			<xacro:property name="connected_to" value="${arm_parent_link if arm_parent_link else default_parent_link}" />
-			<xacro:property name="dof" value="${arm_cfg.get('dof', 6)}" />
-			<xacro:zlab_robot_arm arm_id="${arm_id}"
-				prefix="${prefix}"
-				connected_to="${connected_to}"
-				base_xyz="${base_xyz_str}"
-				base_rpy="${base_rpy_str}"
-				dof="${dof}" />
-			<xacro:property name="remaining_arms" value="${arm_list[1:]}" />
-			<xacro:instantiate_arms arm_list="${remaining_arms}" />
-		</xacro:if>
-	</xacro:macro>
-	<!-- Gazebo 传动宏 -->
-	<xacro:macro name="gazebo-joint" params="joint ">
-		<transmission name="trans_${joint}">
-			<type>transmission_interface/SimpleTransmission</type>
-			<joint name="${joint}">
-				<hardwareInterface>hardware_interface/PositionJointInterface</hardwareInterface>
-			</joint>
-			<actuator name="${joint}_motor">
-				<hardwareInterface>hardware_interface/PositionJointInterface</hardwareInterface>
-				<mechanicalReduction>1</mechanicalReduction>
-			</actuator>
-		</transmission>
-	</xacro:macro>
-	<!-- 机械臂宏定义 -->
-		<xacro:macro name="zlab_robot_arm" params="arm_id:='zlab_arm' prefix:='' connected_to:='' base_xyz:='0 0 0' base_rpy:='0 0 0' dof:=6">
-		<xacro:property name="raw_prefix" value="${prefix if prefix != '' else arm_id}" />
-		<xacro:property name="name_prefix" value="${raw_prefix if raw_prefix.endswith('_') else raw_prefix + '_'}" />
-		<xacro:unless value="${connected_to == ''}">
-			<joint name="${name_prefix}joint_base" type="fixed">
-				<parent link="${connected_to}" />
-				<child link="${name_prefix}base0_link" />
-				<origin xyz="${base_xyz}" rpy="${base_rpy}" />
-			</joint>
-		</xacro:unless>
-		<xacro:link_with_inertial name="${name_prefix}base0_link"
-			xyz="0.00022281 -3.2078E-06 0.11314"
-			rpy="0 0 0"
-			mass="50.058"
-			ixx="0.87603"
-			ixy="-2.9247E-05"
-			ixz="9.7148E-05"
-			iyy="0.87602"
-			iyz="-1.6883E-06"
-			izz="1.5353"
-			visual_mesh="package://zlab_robot_description/meshes/collision/extra_base_link.STL"
-			collision_mesh="package://zlab_robot_description/meshes/collision/extra_base_link.STL" />
-		<xacro:link_with_inertial name="${name_prefix}base1_link"
-			xyz="2.7756E-16 2.2204E-16 -0.008"
-			rpy="0 0 0"
-			mass="3.1592"
-			ixx="0.0064529"
-			ixy="-1.9807E-18"
-			ixz="1.3186E-21"
-			iyy="0.0064529"
-			iyz="-1.7017E-21"
-			izz="0.012771"
-			visual_mesh="package://zlab_robot_description/meshes/collision/plant_link.STL"
-			collision_mesh="package://zlab_robot_description/meshes/collision/plant_link.STL" />
-		<joint name="${name_prefix}base0_to_base1" type="fixed">
-			<parent link="${name_prefix}base0_link" />
-			<child link="${name_prefix}base1_link" />
-			<origin xyz="0 0 0.487" rpy="0 0 0" />
-		</joint>
-		<xacro:link_with_inertial name="${name_prefix}base2_link"
-			xyz="-0.00031896 -0.00029673 0.042463"
-			rpy="0 0 0"
-			mass="1.6185"
-			ixx="0.0030836"
-			ixy="1.5354E-05"
-			ixz="-1.9315E-05"
-			iyy="0.0030825"
-			iyz="-1.7918E-05"
-			izz="0.0045209"
-			visual_mesh="package://zlab_robot_description/meshes/visual/base_link.DAE"
-			collision_mesh="package://zlab_robot_description/meshes/collision/base_link.STL" />
-		<joint name="${name_prefix}base1_to_base2" type="fixed">
-			<parent link="${name_prefix}base1_link" />
-			<child link="${name_prefix}base2_link" />
-			<origin xyz="0 0 0.0001" rpy="0 0 0" />
-		</joint>
-		<xacro:link_with_inertial name="${name_prefix}j1_link"
-			xyz="5.0029E-07 -0.0040922 0.14629"
-			rpy="0 0 0"
-			mass="4.3771"
-			ixx="0.010731"
-			ixy="-8.0587E-09"
-			ixz="-3.6773E-08"
-			iyy="0.010408"
-			iyz="0.00012853"
-			izz="0.0081793"
-			visual_mesh="package://zlab_robot_description/meshes/visual/j1_link.DAE"
-			collision_mesh="package://zlab_robot_description/meshes/collision/j1_link.STL" />
-		<joint name="${name_prefix}j1" type="revolute">
-			<origin xyz="0 0 0" rpy="0 0 0" />
-			<parent link="${name_prefix}base2_link" />
-			<child link="${name_prefix}j1_link" />
-			<axis xyz="0 0 1" />
-			<limit lower="-3.0543" upper="3.0543" effort="150" velocity="3.15" />
-			<calibration rising="0" falling="0" />
-			<dynamics damping="0" friction="0" />
-			<safety_controller soft_lower_limit="-3.0543" soft_upper_limit="3.0543" k_position="15" k_velocity="10" />
-		</joint>
-		<xacro:gazebo-joint joint="${name_prefix}j1" />
-		<xacro:link_with_inertial name="${name_prefix}j2_link"
-			xyz="-0.2125 -5.7643E-09 0.1346"
-			rpy="0 0 0"
-			mass="14.458"
-			ixx="0.028392"
-			ixy="-1.337E-07"
-			ixz="-3.9895E-09"
-			iyy="0.4559"
-			iyz="4.214E-08"
-			izz="0.44974"
-			visual_mesh="package://zlab_robot_description/meshes/visual/j2_link.DAE"
-			collision_mesh="package://zlab_robot_description/meshes/collision/j2_link.STL" />
-		<joint name="${name_prefix}j2" type="revolute">
-			<origin xyz="0 0 0.152" rpy="1.5708 0 0" />
-			<parent link="${name_prefix}j1_link" />
-			<child link="${name_prefix}j2_link" />
-			<axis xyz="0 0 1" />
-			<limit lower="-4.6251" upper="1.4835" effort="150" velocity="3.15" />
-			<calibration rising="0" falling="0" />
-			<dynamics damping="0" friction="0" />
-			<safety_controller soft_lower_limit="-4.6251" soft_upper_limit="1.4835" k_position="15" k_velocity="10" />
-		</joint>
-		<xacro:gazebo-joint joint="${name_prefix}j2" />
-		<xacro:link_with_inertial name="${name_prefix}j3_link"
-			xyz="-0.18793 -8.4503E-07 0.0066357"
-			rpy="0 0 0"
-			mass="7.6737"
-			ixx="0.0085096"
-			ixy="2.1613E-06"
-			ixz="-0.0068678"
-			iyy="0.16971"
-			iyz="3.7086E-08"
-			izz="0.16854"
-			visual_mesh="package://zlab_robot_description/meshes/visual/j3_link.DAE"
-			collision_mesh="package://zlab_robot_description/meshes/collision/j3_link.STL" />
-		<joint name="${name_prefix}j3" type="revolute">
-			<origin xyz="-0.425 0 0" rpy="0 0 0" />
-			<parent link="${name_prefix}j2_link" />
-			<child link="${name_prefix}j3_link" />
-			<axis xyz="0 0 1" />
-			<limit lower="-2.8274" upper="2.8274" effort="150" velocity="3.15" />
-			<calibration rising="0" falling="0" />
-			<dynamics damping="0" friction="0" />
-			<safety_controller soft_lower_limit="-2.8274" soft_upper_limit="2.8274" k_position="15" k_velocity="10" />
-		</joint>
-		<xacro:gazebo-joint joint="${name_prefix}j3" />
-		<xacro:link_with_inertial name="${name_prefix}j4_link"
-			xyz="4.98E-07 -0.003754 0.097155"
-			rpy="0 0 0"
-			mass="1.6266"
-			ixx="0.00216"
-			ixy="4.888E-09"
-			ixz="3.1528E-08"
-			iyy="0.0015455"
-			iyz="3.7678E-05"
-			izz="0.0019902"
-			visual_mesh="package://zlab_robot_description/meshes/visual/j4_link.DAE"
-			collision_mesh="package://zlab_robot_description/meshes/collision/j4_link.STL" />
-		<joint name="${name_prefix}j4" type="revolute">
-			<origin xyz="-0.39501 0 0" rpy="0 0 0" />
-			<parent link="${name_prefix}j3_link" />
-			<child link="${name_prefix}j4_link" />
-			<axis xyz="0 0 1" />
-			<limit lower="-4.6251" upper="1.4835" effort="28" velocity="3.2" />
-			<calibration rising="0" falling="0" />
-			<dynamics damping="0" friction="0" />
-			<safety_controller soft_lower_limit="-4.6251" soft_upper_limit="1.4835" k_position="15" k_velocity="10" />
-		</joint>
-		<xacro:gazebo-joint joint="${name_prefix}j4" />
-		<xacro:link_with_inertial name="${name_prefix}j5_link"
-			xyz="-4.5588E-07 0.0038617 0.098257"
-			rpy="0 0 0"
-			mass="1.5812"
-			ixx="0.0020612"
-			ixy="8.7064E-09"
-			ixz="-3.4742E-08"
-			iyy="0.0014477"
-			iyz="-2.8534E-05"
-			izz="0.0019573"
-			visual_mesh="package://zlab_robot_description/meshes/visual/j5_link.DAE"
-			collision_mesh="package://zlab_robot_description/meshes/collision/j5_link.STL" />
-		<joint name="${name_prefix}j5" type="revolute">
-			<origin xyz="0 0 0.1021" rpy="1.5708 0 0" />
-			<parent link="${name_prefix}j4_link" />
-			<child link="${name_prefix}j5_link" />
-			<axis xyz="0 0 1" />
-			<limit lower="-3.0543" upper="3.0543" effort="28" velocity="3.2" />
-			<calibration rising="0" falling="0" />
-			<dynamics damping="0" friction="0" />
-			<safety_controller soft_lower_limit="-3.0543" soft_upper_limit="3.0543" k_position="15" k_velocity="10" />
-		</joint>
-		<xacro:gazebo-joint joint="${name_prefix}j5" />
-		<xacro:link_with_inertial name="${name_prefix}j6_link"
-			xyz="7.7496E-05 1.7751E-05 0.076122"
-			rpy="0 0 0"
-			mass="0.52542"
-			ixx="0.00027721"
-			ixy="-1.8677E-09"
-			ixz="-1.188E-07"
-			iyy="0.00027839"
-			iyz="2.2607E-07"
-			izz="0.00041605"
-			visual_mesh="package://zlab_robot_description/meshes/visual/j6_link.DAE"
-			collision_mesh="package://zlab_robot_description/meshes/collision/j6_link.STL" />
-		<joint name="${name_prefix}j6" type="revolute">
-			<origin xyz="0 0 0.102" rpy="-1.5708 0 0" />
-			<parent link="${name_prefix}j5_link" />
-			<child link="${name_prefix}j6_link" />
-			<axis xyz="0 0 1" />
-			<limit lower="-3.0543" upper="3.0543" effort="28" velocity="3.2" />
-			<calibration rising="0" falling="0" />
-			<dynamics damping="0" friction="0" />
-			<safety_controller soft_lower_limit="-3.0543" soft_upper_limit="3.0543" k_position="15" k_velocity="10" />
-		</joint>
-		<xacro:gazebo-joint joint="${name_prefix}j6" />
-	</xacro:macro>
-	<!-- 顶层结构 -->
-	<link name="world" />
-	<xacro:if value="${len(enabled_arms) == 0}">
-		<xacro:property name="raw_fallback_prefix" value="${default_prefix if default_prefix != '' else arm_id}" />
-		<xacro:property name="fallback_prefix" value="${raw_fallback_prefix if raw_fallback_prefix.endswith('_') else raw_fallback_prefix + '_'}" />
-		<xacro:zlab_robot_arm arm_id="$(arg arm_id)"
-			prefix="${fallback_prefix}"
-			connected_to="${default_parent_link}"
-			base_xyz="$(arg base_xyz)"
-			base_rpy="$(arg base_rpy)" />
-	</xacro:if>
-	<xacro:instantiate_arms arm_list="${enabled_arms}" />
-	<gazebo>
-		<plugin name="gazebo_ros_control" filename="libgazebo_ros_control.so" />
-	</gazebo>
+    <!-- 机械臂配置参数 -->
+    <xacro:arg name="config_file" default="" />
+    <!-- 配置文件加载和解析 -->
+    <xacro:property name="robot_config" value="${xacro.load_yaml('$(arg config_file)')}" />
+    <xacro:property name="arms_config" value="${robot_config['arms']}" />
+    <xacro:property name="enabled_arms"
+        value="${[(name, cfg) for name, cfg in arms_config.items() if cfg.get('enabled', False)]}" />
+    <!-- 通用外观设置 -->
+    <xacro:property name="link_material" value="silver" />
+    <xacro:property name="link_color_rgba" value="0.89804 0.91765 0.92941 1" />
+    <!-- 材质定义宏 -->
+    <xacro:macro name="robot_material" params="name rgba:='${link_color_rgba}'">
+        <material name="${name}">
+            <color rgba="${rgba}" />
+        </material>
+    </xacro:macro>
+    <!-- 可复用的带惯量链接定义 -->
+    <xacro:macro name="link_with_inertial"
+        params="name xyz rpy mass ixx ixy ixz iyy iyz izz visual_mesh collision_mesh
+                scale:='1 1 1' material:='${link_material}' color:='${link_color_rgba}'
+                visual_origin_xyz:='0 0 0' visual_origin_rpy:='0 0 0'
+                collision_origin_xyz:='0 0 0' collision_origin_rpy:='0 0 0'">
+        <link name="${name}">
+            <!-- 惯量属性 -->
+            <inertial>
+                <origin xyz="${xyz}" rpy="${rpy}" />
+                <mass value="${mass}" />
+                <inertia ixx="${ixx}" ixy="${ixy}" ixz="${ixz}"
+                    iyy="${iyy}" iyz="${iyz}" izz="${izz}" />
+            </inertial>
+            <!-- 可视化几何体 -->
+            <visual>
+                <origin xyz="${visual_origin_xyz}" rpy="${visual_origin_rpy}" />
+                <geometry>
+                    <mesh filename="${visual_mesh}" scale="${scale}" />
+                </geometry>
+                <material name="${material}">
+                    <color rgba="${color}" />
+                </material>
+            </visual>
+            <!-- 碰撞几何体 -->
+            <collision>
+                <origin xyz="${collision_origin_xyz}" rpy="${collision_origin_rpy}" />
+                <geometry>
+                    <mesh filename="${collision_mesh}" scale="${scale}" />
+                </geometry>
+            </collision>
+        </link>
+    </xacro:macro>
+    <xacro:macro name="instantiate_arms" params="arm_list">
+        <xacro:if value="${len(arm_list) > 0}">
+            <xacro:property name="arm_entry" value="${arm_list[0]}" />
+            <xacro:property name="arm_cfg" value="${arm_entry[1]}" />
+            <xacro:property name="arm_name" value="${arm_entry[0]}" />
+            <xacro:property name="arm_id" value="${arm_cfg.get('arm_id', arm_name)}" />
+            <xacro:property name="raw_prefix" value="${arm_cfg.get('prefix', arm_name)}" />
+            <xacro:property name="prefix"
+                value="${raw_prefix if raw_prefix.endswith('_') else raw_prefix + '_'}" />
+            <xacro:property name="base_xyz_list" value="${arm_cfg.get('base_xyz', [0.0, 0.0, 0.0])}" />
+            <xacro:property name="base_rpy_list" value="${arm_cfg.get('base_rpy', [0.0, 0.0, 0.0])}" />
+            <xacro:property name="base_xyz_str" value="${' '.join([str(x) for x in base_xyz_list])}" />
+            <xacro:property name="base_rpy_str" value="${' '.join([str(x) for x in base_rpy_list])}" />
+            <xacro:property name="arm_parent_link" value="${arm_cfg.get('parent_link', 'world')}" />
+            <xacro:property name="dof" value="${arm_cfg.get('dof', 6)}" />
+            <xacro:zlab_robot_arm
+                arm_id="${arm_id}"
+                prefix="${prefix}"
+                connected_to="${arm_parent_link}"
+                base_xyz="${base_xyz_str}"
+                base_rpy="${base_rpy_str}"
+                dof="${dof}" />
+            <xacro:property name="remaining_arms" value="${arm_list[1:]}" />
+            <xacro:instantiate_arms arm_list="${remaining_arms}" />
+        </xacro:if>
+    </xacro:macro>
+    <!-- Gazebo 传动宏 -->
+    <xacro:macro name="gazebo_joint_transmission"
+        params="joint_name reduction:=1 interface:='hardware_interface/PositionJointInterface'">
+        <transmission name="trans_${joint_name}">
+            <type>transmission_interface/SimpleTransmission</type>
+            <joint name="${joint_name}">
+                <hardwareInterface>${interface}</hardwareInterface>
+            </joint>
+            <actuator name="${joint_name}_motor">
+                <hardwareInterface>${interface}</hardwareInterface>
+                <mechanicalReduction>${reduction}</mechanicalReduction>
+            </actuator>
+        </transmission>
+    </xacro:macro>
+    <!-- 向后兼容的传动宏 -->
+    <xacro:macro name="gazebo-joint" params="joint">
+        <xacro:gazebo_joint_transmission joint_name="${joint}" />
+    </xacro:macro>
+    <!-- 机械臂宏定义 -->
+    <xacro:macro name="zlab_robot_arm"
+        params="arm_id:='zlab_arm' prefix:='' connected_to:='' base_xyz:='0 0 0' base_rpy:='0 0 0' dof:=6">
+        <xacro:property name="raw_prefix" value="${prefix if prefix != '' else arm_id}" />
+        <xacro:property name="name_prefix"
+            value="${raw_prefix if raw_prefix.endswith('_') else raw_prefix + '_'}" />
+        <xacro:unless value="${connected_to == ''}">
+            <joint name="${name_prefix}joint_base" type="fixed">
+                <parent link="${connected_to}" />
+                <child link="${name_prefix}base0_link" />
+                <origin xyz="${base_xyz}" rpy="${base_rpy}" />
+            </joint>
+        </xacro:unless>
+        <xacro:link_with_inertial name="${name_prefix}base0_link"
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
Commit message: 20251010 增加end_effector

File: src/zlab_robot_description/urdf/zlab_robot.urdf.xacro (robot description, xacro)
@@ -297,4 +297,13 @@
         </joint>
         <xacro:gazebo-joint joint="${name_prefix}j6" />
+        <!-- End effector link for proper tool positioning -->
+        <link name="${name_prefix}end_effector">
+            <!-- Empty link for end effector reference frame -->
+        </link>
+        <joint name="${name_prefix}end_effector_joint" type="fixed">
+            <origin xyz="0 0 0.07" rpy="0 0 0" />
+            <parent link="${name_prefix}j6_link" />
+            <child link="${name_prefix}end_effector" />
+        </joint>
     </xacro:macro>
     <!-- 顶层结构 -->

File: src/zlab_robot_description/urdf/zlab_robot_dual_arm.urdf (robot description, URDF)
Before this commit: robot zlab_robot, 19 links, 18 joints
Links:
- added link l_end_effector
- added link r_end_effector
Joints:
- added joint l_end_effector_joint: type fixed, parent l_j6_link, child l_end_effector, origin xyz=0 0 0.07 rpy=0 0 0
- added joint r_end_effector_joint: type fixed, parent r_j6_link, child r_end_effector, origin xyz=0 0 0.07 rpy=0 0 0

File: src/zlab_robot_description/urdf/zlab_robot_single_arm.urdf (robot description, URDF)
Before this commit: robot zlab_robot, 10 links, 9 joints
Links:
- added link zlab_arm_end_effector
Joints:
- added joint zlab_arm_end_effector_joint: type fixed, parent zlab_arm_j6_link, child zlab_arm_end_effector, origin xyz=0 0 0.07 rpy=0 0 0

Commit message: 20251010 MoveIt single 配置完成

File: src/zlab_robot_description/urdf/zlab_robot.urdf.xacro (robot description, xacro)
@@ -297,13 +297,4 @@
         </joint>
         <xacro:gazebo-joint joint="${name_prefix}j6" />
-        <!-- End effector link for proper tool positioning -->
-        <link name="${name_prefix}end_effector">
-            <!-- Empty link for end effector reference frame -->
-        </link>
-        <joint name="${name_prefix}end_effector_joint" type="fixed">
-            <origin xyz="0 0 0.07" rpy="0 0 0" />
-            <parent link="${name_prefix}j6_link" />
-            <child link="${name_prefix}end_effector" />
-        </joint>
     </xacro:macro>
     <!-- 顶层结构 -->
