Commit message: 20251011

File: src/zlab_robot_description/urdf/zlab_robot.urdf.xacro (robot description, xacro)
@@ -297,4 +297,19 @@
         </joint>
         <xacro:gazebo-joint joint="${name_prefix}j6" />
+        <!-- Tool0 link - 末端执行器参考点 -->
+        <link name="${name_prefix}tool0">
+            <inertial>
+                <origin xyz="0 0 0" rpy="0 0 0" />
+                <mass value="0.001" />
+                <inertia ixx="0.000001" ixy="0" ixz="0"
+                    iyy="0.000001" iyz="0" izz="0.000001" />
+            </inertial>
+        </link>
+        <!-- Tool0 joint - 连接 j6_link 到 tool0 -->
+        <joint name="${name_prefix}j6_tool0" type="fixed">
+            <origin xyz="0 0 0.1" rpy="0 0 0" />
+            <parent link="${name_prefix}j6_link" />
+            <child link="${name_prefix}tool0" />
+        </joint>
     </xacro:macro>
     <!-- 顶层结构 -->

File: src/zlab_robot_description/urdf/zlab_robot_dual_arm.urdf.xacro (robot description, xacro)
@@ -7,5 +7,11 @@
     <!-- 指定配置文件 -->
     <xacro:arg name="config_file" default="$(find zlab_robot_description)/config/robot_config_dual_arm.yaml" />
+    <!-- 初始位置文件 -->
+    <xacro:arg name="initial_positions_file" default="$(find zlab_robot_moveit_config)/config/dual_arm/initial_positions.yaml" />
     <!-- 引入主 xacro 文件 -->
     <xacro:include filename="$(find zlab_robot_description)/urdf/zlab_robot.urdf.xacro" />
+    <!-- 引入 ros2_control 配置 -->
+    <xacro:include filename="$(find zlab_robot_moveit_config)/config/dual_arm/zlab_robot_dual_arm.ros2_control.xacro" />
+    <!-- 实例化 ros2_control -->
+    <xacro:zlab_robot_dual_arm_ros2_control name="FakeSystem" initial_positions_file="$(arg initial_positions_file)"/>
 </robot>

File: src/zlab_robot_description/urdf/zlab_robot_single_arm.urdf.xacro (robot description, xacro)
@@ -7,5 +7,11 @@
     <!-- 指定配置文件 -->
     <xacro:arg name="config_file" default="$(find zlab_robot_description)/config/robot_config_single_arm.yaml" />
+    <!-- 初始位置文件 -->
+    <xacro:arg name="initial_positions_file" default="$(find zlab_robot_moveit_config)/config/single_arm/initial_positions.yaml" />
     <!-- 引入主 xacro 文件 -->
     <xacro:include filename="$(find zlab_robot_description)/urdf/zlab_robot.urdf.xacro" />
+    <!-- 引入 ros2_control 配置 -->
+    <xacro:include filename="$(find zlab_robot_moveit_config)/config/single_arm/zlab_robot_single_arm.ros2_control.xacro" />
+    <!-- 实例化 ros2_control -->
+    <xacro:zlab_robot_single_arm_ros2_control name="FakeSystem" initial_positions_file="$(arg initial_positions_file)"/>
 </robot>

Commit message: 20251014 解决moveit崩溃问题

File: src/zlab_robot_description/urdf/zlab_robot.urdf.xacro (robot description, xacro)
@@ -97,7 +97,7 @@
     <xacro:macro name="zlab_robot_arm"
         params="arm_id:='zlab_arm' prefix:='' connected_to:='' base_xyz:='0 0 0' base_rpy:='0 0 0' dof:=6">
-        <xacro:property name="raw_prefix" value="${prefix if prefix != '' else arm_id}" />
+        <!-- 修改前缀逻辑：prefix为空则不加前缀 -->
         <xacro:property name="name_prefix"
-            value="${raw_prefix if raw_prefix != '' and raw_prefix.endswith('_') else (raw_prefix + '_' if raw_prefix != '' else '')}" />
+            value="${prefix if prefix != '' else ''}" />
         <xacro:unless value="${connected_to == ''}">
             <joint name="${name_prefix}joint_base" type="fixed">
@@ -297,4 +297,22 @@
         </joint>
         <xacro:gazebo-joint joint="${name_prefix}j6" />
+        <!-- 末端虚拟链接 -->
+        <link name="${name_prefix}ee_link">
+            <inertial>
+                <mass value="0.01"/>
+                <inertia ixx="0.0001" ixy="0.0" ixz="0.0" iyy="0.0001" iyz="0.0" izz="0.0001"/>
+            </inertial>
+        </link>
+        <joint name="${name_prefix}j6_to_ee" type="fixed">
+            <parent link="${name_prefix}j6_link" />
+            <child link="${name_prefix}ee_link" />
+            <origin xyz="0 0 0.1" rpy="0 0 0" />
+        </joint>
+        <!-- Gazebo 设置，防止关节合并 -->
+        <gazebo reference="${name_prefix}j6_to_ee">
+            <preserveFixedJoint>true</preserveFixedJoint>
+            <!-- For compatibility with SDFormat < 4.4 -->
+            <disableFixedJointLumping>true</disableFixedJointLumping>
+        </gazebo>
     </xacro:macro>
     <!-- 顶层结构 -->

File: src/zlab_robot_description/urdf/zlab_robot_dual_arm.urdf.xacro (robot description, xacro)
@@ -4,5 +4,5 @@
     这是一个包装文件，引用主 xacro 并指定双臂配置
 -->
-<robot xmlns:xacro="http://www.ros.org/wiki/xacro" name="zlab_robot_dual_arm">
+<robot xmlns:xacro="http://www.ros.org/wiki/xacro" name="dual_arm">
     <!-- 指定配置文件 -->
     <xacro:arg name="config_file" default="$(find zlab_robot_description)/config/robot_config_dual_arm.yaml" />

File: src/zlab_robot_description/urdf/zlab_robot_single_arm.urdf.xacro (robot description, xacro)
@@ -4,5 +4,5 @@
     这是一个包装文件，引用主 xacro 并指定单臂配置
 -->
-<robot xmlns:xacro="http://www.ros.org/wiki/xacro" name="zlab_robot_single_arm">
+<robot xmlns:xacro="http://www.ros.org/wiki/xacro" name="single_arm">
     <!-- 指定配置文件 -->
     <xacro:arg name="config_file" default="$(find zlab_robot_description)/config/robot_config_single_arm.yaml" />
